File: SOURCES/KICAD/AnalogIO-x8.kicad_pcb (KiCad board)
At the start: 2 copper layers, 120 x 120 mm, 418 parts, among them IC101 IC_TLE2426ID, IC102 IC_ADM811TARTZ, IC103 IC_LM1117MP-5.0, IC104 IC_LM1117MPX-ADJ, IC105 IC_NCP1117LPST33, IC201 IC_NE5532AD_SOIC8, IC202 IC_NE5532AD_SOIC8, IC203 IC_NE5532AD_SOIC8, IC204 IC_NE5532AD_SOIC8, IC205 IC_AK5558VN, IC206 IC_NE5532AD_SOIC8, IC207 IC_NE5532AD_SOIC8, IC208 IC_NE5532AD_SOIC8, IC209 IC_NE5532AD_SOIC8, IC301 IC_NE5532AD_SOIC8, IC302 IC_NE5532AD_SOIC8, IC303 IC_NE5532AD_SOIC8, IC304 IC_NE5532AD_SOIC8, IC305 IC_AK4458VN, IC306 IC_NE5532AD_SOIC8, IC307 IC_NE5532AD_SOIC8, IC308 IC_NE5532AD_SOIC8, IC309 IC_NE5532AD_SOIC8, X101 CON_IDC64, X102 CON_IDC64, X103 CON_MicroFit3_02x02, X104 CON_MicroFit3_02x02, X201 CON_IDC26, X202 CON_DSUB25F, X301 CON_DSUB25F, X302 CON_IDC26

Commit message: Created Gerbers and BOM
Other:
- board text added: "auverdion AnalogIO-x8"
- board text removed: "auverdion ai8o8"
Changed lines of the file:
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@@
     (links 993)
     (no_connects 0)
-    (area 79.924999 29.924999 200.075001 150.075001)
+    (area 70.714266 23.972599 202.02383 150.100001)
     (thickness 1.6)
     (drawings 11)
@@
     (effects (font (size 1.5 1.5) (thickness 0.3)))
   )
-  (gr_text "auverdion\nai8o8" (at 148 121) (layer F.SilkS)
+  (gr_text "auverdion\nAnalogIO-x8" (at 148 121) (layer F.SilkS)
     (effects (font (size 2 2) (thickness 0.3)))
   )
@@
         (xy 80 30) (xy 200 30) (xy 200 109.5) (xy 178.5 109.5) (xy 178.5 103.8)
         (xy 157.8 103.8) (xy 157.8 108.9) (xy 127.4 108.9) (xy 121.4 108.9) (xy 119.8 110.5)
-        (xy 98.3 110.5) (xy 92.7 116.1) (xy 80 116.1)
+        (xy 100.4 110.5) (xy 90.9 120) (xy 80 120)
       )
     )
