File: SOURCES/KICAD/AnalogIO-x8.sch (KiCad schematic (older format))
At the start: 38 parts, among them IC101 IC_TLE2426ID, IC102 IC_ADM811TARTZ, IC103 IC_LM1117MP-5.0, IC104 IC_LM1117MPX-ADJ, IC105 IC_NCP1117LPST33, X101 CON_IDC64, X102 CON_IDC64, X103 CON_MicroFit3_02x02, X104 CON_MicroFit3_02x02

Commit message: Added some comments to schematics
Parts:
- C101, C104, C107, C116: symbol CAP_100n_50V_X7R_0805 -> rk:CAP_100n_50V_X7R_0805
- C102, C103, C105, C106, C108, C115, C117, C118: symbol CAP_10u0_25V_X5R_0805 -> rk:CAP_10u0_25V_X5R_0805
- C109, C110, C111, C112, C113, C114: symbol CAP_100u_20%_25V_ALUM_RADIAL -> rk:CAP_100u_20%_25V_ALUM_RADIAL
- D101: symbol D -> Device:D
- IC101: symbol IC_TLE2426ID -> rk:IC_TLE2426ID
- IC102: symbol IC_ADM811TARTZ -> rk:IC_ADM811TARTZ
- IC103: symbol IC_LM1117MP-5.0 -> rk:IC_LM1117MP-5.0
- IC104: symbol IC_LM1117MPX-ADJ -> rk:IC_LM1117MPX-ADJ
- IC105: symbol IC_NCP1117LPST33 -> rk:IC_NCP1117LPST33
- R101: symbol RES_100K_1%_0.125W_Thick_0805 -> rk:RES_100K_1%_0.125W_Thick_0805
- R102, R105: symbol R -> Device:R
- R103: symbol RES_150R_1%_0.25W_Thin_0805 -> rk:RES_150R_1%_0.25W_Thin_0805
- R104: symbol RES_931R_1%_0.125W_Thick_0805 -> rk:RES_931R_1%_0.125W_Thick_0805
- X101, X102: symbol CON_IDC64 -> rk:CON_IDC64
- X103, X104: symbol CON_MicroFit3_02x02 -> rk:CON_MicroFit3_02x02
Connections:
- net +12V: no longer IC105.3 (IN)
- net +9V: no longer IC104.4 (OUT)

Commit message: Documentation
Parts:
- B101, B102, B103, B104, B105: symbol TEST_1P -> Connector:TestPoint
Connections:
- wire segments 275 -> 276
Other:
- note added: "Single Supply Option"
- moved on the sheet: C101, C102, C103, C104, C105, C106, C107, C108, C109, C110, C111, C118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
