File: SOURCES/KICAD/adc.sch (KiCad schematic (older format))
At the start: 216 parts, among them IC201 IC_NE5532AD_SOIC8, IC202 IC_NE5532AD_SOIC8, IC203 IC_NE5532AD_SOIC8, IC204 IC_NE5532AD_SOIC8, IC205 IC_AK5558VN, IC206 IC_NE5532AD_SOIC8, IC207 IC_NE5532AD_SOIC8, IC208 IC_NE5532AD_SOIC8, IC209 IC_NE5532AD_SOIC8, X201 CON_IDC26, X202 CON_DSUB25F

Commit message: Added some comments to schematics
Parts:
- C201, C202, C211, C212, C219, C220, C231, C232, C241, C242, C253, C254, C265, C266, C275, C276: symbol CAP_1n00_5%_50V_PPS_0805 -> rk:CAP_1n00_5%_50V_PPS_0805
- C203, C204, C213, C214, C221, C222, C227, C233, C234, C239, C243, C244, C245, C255, C256, C257, C267, C268, C283, C284: symbol CAP_100u_20%_25V_ALUM_RADIAL -> rk:CAP_100u_20%_25V_ALUM_RADIAL
- C205, C206, C215, C216, C223, C224, C235, C236, C247, C248, C259, C260, C269, C270, C285, C286: symbol CAP_1n00_50V_X7R_0805 -> rk:CAP_1n00_50V_X7R_0805
- C207, C208, C217, C218, C225, C226, C237, C238, C249, C250, C261, C262, C271, C272, C287, C288: symbol CAP_100p_50V_C0G/NP0_0805 -> rk:CAP_100p_50V_C0G_NP0_0805
- C209, C210, C229, C230, C251, C252, C273, C274: symbol CAP_5n60_5%_16V_PPS_0805 -> rk:CAP_5n60_5%_16V_PPS_0805
- C228, C240, C246, C258, C263, C279, C280, C282, C289, C290, C291, C292, C293, C294, C295, C296, C297, C298, C299, C300, C301, C302, C303, C304: symbol CAP_100n_50V_X7R_0805 -> rk:CAP_100n_50V_X7R_0805
- C264: symbol CAP_4u70_25V_X5R_0805 -> rk:CAP_4u70_25V_X5R_0805
- C277, C278: symbol CAP_10u0_25V_X5R_0805 -> rk:CAP_10u0_25V_X5R_0805
- C281: symbol CAP_10n0_50V_X7R_0805 -> rk:CAP_10n0_50V_X7R_0805
- IC201, IC202, IC203, IC204, IC206, IC207, IC208, IC209: symbol IC_NE5532AD_SOIC8 -> rk:IC_NE5532AD_SOIC8
- IC205: symbol IC_AK5558VN -> rk:IC_AK5558VN
- R201, R202, R211, R212, R221, R222, R240, R241, R255, R256, R267, R268, R277, R278, R287, R288: symbol RES_620R_0.5%_0.1W_Thin_0805 -> rk:RES_620R_0.5%_0.1W_Thin_0805
- R203, R205, R213, R215, R223, R225, R242, R244, R257, R259, R269, R271, R279, R281, R289, R291: symbol RES_100R_1%_0.25W_Thin_0805 -> rk:RES_100R_1%_0.25W_Thin_0805
- R204, R206, R214, R216, R224, R226, R243, R245, R258, R260, R270, R272, R280, R282, R290, R292: symbol RES_976R_0.5%_0.1W_Thin_0805 -> rk:RES_976R_0.5%_0.1W_Thin_0805
- R207, R208, R217, R218, R227, R228, R246, R247, R262, R263, R273, R274, R283, R284, R293, R294: symbol RES_10R0_1%_0.25W_Thin_0805 -> rk:RES_10R0_1%_0.25W_Thin_0805
- R209, R210, R219, R220, R234, R235, R248, R249, R264, R265, R275, R276, R285, R286, R295, R296: symbol RES_100K_1%_0.125W_Thick_0805 -> rk:RES_100K_1%_0.125W_Thick_0805
- R229, R231, R233, R251, R252, R253, R297, R299, R300, R375: symbol RES_0R00_1%_0.125W_Thick_0805 -> rk:RES_0R00_1%_0.125W_Thick_0805
- R230, R232, R237, R238, R239, R298: symbol RES_47K0_1%_0.125W_Thick_0805 -> rk:RES_47K0_1%_0.125W_Thick_0805
- R236, R250, R254, R266: symbol RES_20R0_1%_0.125W_Thick_0805 -> rk:RES_20R0_1%_0.125W_Thick_0805
- R261: symbol RES_51R0_1%_0.125W_Thick_0805 -> rk:RES_51R0_1%_0.125W_Thick_0805
- X201: symbol CON_IDC26 -> rk:CON_IDC26
- X202: symbol CON_DSUB25F -> rk:CON_DSUB25F
Connections:
- wire segments 423 -> 608
Other:
- note added: "For Infinitas:\nR251, R252, R300, R375: 0R00\nR237, R239: 47K0\nR238, R253: DNP"
- note added: "R231, R233, R297, R299: 0R00\nR230: 47K0\nR232, R298: DNP"

Commit message: Documentation
Other:
- note added: "For Infinitas:\nR231, R233, R251, R252, \nR297, R299, R300, R375: 0R00\nR230, R237, R239: 47K0\nR232, R238, R253, R298: DNP\n\nSee datasheet for other configurations.\nRemove R300 and R301 for hardware mode\n(parallel mode)."
- note added: "I2C Addr: 0x22/0x23"
- note removed: "Addr: 0x22/0x23"
- note removed: "For Infinitas:\nR251, R252, R300, R375: 0R00\nR237, R239: 47K0\nR238, R253: DNP"
- note removed: "R231, R233, R297, R299: 0R00\nR230: 47K0\nR232, R298: DNP"
- note removed: "alternative OpAmps: OPA1652, OPA2365, OPA2353"
- note removed: "see datasheet for configuration"
Changed lines of the file:
@@
 NoConn ~ 12750 5800
 NoConn ~ 12750 5700
-Text Notes 13150 4100 0    39   ~ 0
-see datasheet for configuration
 Text HLabel 13250 5400 2    39   Output ~ 0
 OVF
@@
 Text HLabel 7000 9000 0    39   Input ~ 0
 VGROUND
-Text Notes 6100 9950 0    60   ~ 0
-alternative OpAmps: OPA1652, OPA2365, OPA2353
 Wire Wire Line
 	1500 7550 1450 7550
@@
 Connection ~ 12800 4000
 Connection ~ 12000 4200
-Text Notes 13150 4250 0    39   ~ 0
-Addr: 0x22/0x23
+Text Notes 14550 4900 0    39   ~ 0
+I2C Addr: 0x22/0x23
 $Comp
 L rk:RES_0R00_1%_0.125W_Thick_0805 R229
@@
 Wire Wire Line
 	12000 4200 12450 4200
-Text Notes 14800 5250 0    39   ~ 0
-For Infinitas:\nR251, R252, R300, R375: 0R00\nR237, R239: 47K0\nR238, R253: DNP
-Text Notes 12600 3550 0    39   ~ 0
-R231, R233, R297, R299: 0R00\nR230: 47K0\nR232, R298: DNP
+Text Notes 14550 4750 0    39   ~ 0
+For Infinitas:\nR231, R233, R251, R252, \nR297, R299, R300, R375: 0R00\nR230, R237, R239:        47K0\nR232, R238, R253, R298: DNP\n\nSee datasheet for other configurations.\nRemove R300 and R301 for hardware mode\n(parallel mode).
 $EndSCHEMATC
