File: SOURCES/KICAD/dac.sch (KiCad schematic (older format))
At the start: 164 parts, among them IC301 IC_NE5532AD_SOIC8, IC302 IC_NE5532AD_SOIC8, IC303 IC_NE5532AD_SOIC8, IC304 IC_NE5532AD_SOIC8, IC305 IC_AK4458VN, IC306 IC_NE5532AD_SOIC8, IC307 IC_NE5532AD_SOIC8, IC308 IC_NE5532AD_SOIC8, IC309 IC_NE5532AD_SOIC8, X301 CON_DSUB25F, X302 CON_IDC26

Commit message: Documentation
Other:
- note added: "For Infinitas\nR359, R360, R376, R377: 0R00\nR364, R365, R374: DNP\n\nSee datasheet for other configurations.\nRemove R376 and R377 for hardware mode\n(parallel mode)."
- note added: "I2C Addr: 0x20/0x21"
- note removed: "Addr: 0x20/0x21"
- note removed: "For Infinitas\nR359, R360, R376, R377: 0R00\nR364, R365, R374: DNP"
- note removed: "See datasheet for configuration"
- note removed: "alternative OpAmps: OPA1652, OPA2365, OPA2353"
Changed lines of the file:
@@
 Wire Wire Line
 	2500 6250 2500 6100
-Text Notes 950  6700 0    39   ~ 0
-See datasheet for configuration
 Wire Wire Line
 	1450 5400 1500 5400
@@
 Wire Wire Line
 	2000 7200 2000 7250
-Text Notes 950  6800 0    39   ~ 0
-Addr: 0x20/0x21
+Text Notes 650  7100 0    39   ~ 0
+I2C Addr: 0x20/0x21
 $Comp
 L rk:RES_0R00_1%_0.125W_Thick_0805 R360
@@
 	1    0    0    -1
 $EndComp
-Text Notes 8350 8200 0    60   ~ 0
-alternative OpAmps: OPA1652, OPA2365, OPA2353
 $Comp
 L rk:IC_AK4458VN IC305
@@
 Wire Wire Line
 	2400 7200 2450 7200
-Text Notes 950  7000 0    39   ~ 0
-For Infinitas\nR359, R360, R376, R377: 0R00\nR364, R365, R374: DNP
+Text Notes 650  6900 0    39   ~ 0
+For Infinitas\nR359, R360, R376, R377: 0R00\nR364, R365, R374: DNP\n\nSee datasheet for other configurations.\nRemove R376 and R377 for hardware mode\n(parallel mode).
 $EndSCHEMATC
